Commit message: Update SO-101 URDF for my camera geometry

File: Simulation/SO101/so101_new_calib.urdf (robot description, URDF)
Before this commit: robot so101_new_calib, 8 links, 7 joints
Links:
- added link camera_link
Joints:
- added joint fixed_camera: type fixed, parent gripper_link, child camera_link, origin xyz=0 0.06620 -0.04905 rpy=0 2.18166 1.5708

Commit message: Change material color

File: Simulation/SO101/so101_new_calib.urdf (robot description, URDF)
Before this commit: robot so101_new_calib, 9 links, 8 joints
Joints:
- joint gripper: limit lower=-0.174533 upper=1.74533 effort=10 velocity=10 -> lower=-0.349066 upper=1.74533 effort=10 velocity=10
